File: PCB/EasyDev-Old/EasyDev-Old.kicad_pcb (KiCad board)
At the start: 2 copper layers, 21 x 51 mm, 35 parts, among them J1 USB_C_Receptacle_USB2.0_14P, J2 Conn_01x20, J3 Conn_01x20, J4 Conn_01x03, J5 Conn_01x01, SW1 SW_Push, U1 RP2040, U2 NCP1117-3.3_SOT223, U3 W25Q128JVS, Y1 12 MHz

Commit message: Uploaded Everything!!
Parts:
- removed D1: WS2812B-2020, LED_SMD:LED_WS2812B-2020_PLCC4_2.0x2.0mm
- removed J5: Conn_01x01, Connector_PinSocket_2.54mm:PinSocket_1x01_P2.54mm_Vertical
Connections:
- U1 pad 37: Net-(D1-DIN) -> unconnected-(U1-GPIO25-Pad37)
Routing:
- net VBUS: track 85.9 -> 25.4 mm, vias 8 -> 0
- net Net-(D1-DIN): track 32.8 -> 0.00 mm, vias 6 -> 0
- net GND: track 111.5 -> 85.2 mm, vias 65 -> 66
- net Net-(D1-DOUT): track 4.95 -> 0.00 mm
- net GPIO20: track 14.5 -> 10.3 mm
- net GPIO29_ADC3: track 33.2 -> 36.2 mm
- net RUN: track 14.4 -> 12.2 mm
- net +3V3: track 117.6 -> 115.6 mm
- net GPIO24: track 16.0 -> 14.1 mm
